File: Flips5X/Flips5X.kicad_pcb (KiCad board)
At the start: 2 copper layers, 100 x 100 mm, 22 parts, among them U1 FP2800A, U2 FP2800A, U3 FP2800A

Commit message: rerouting
Routing:
- net /HV: track 143.5 -> 201.7 mm
- net /SY7: track 126.1 -> 108.5 mm
- net /~RY6: track 81.3 -> 64.8 mm
- net /SY2: track 123.8 -> 111.7 mm
- net /SY5: track 117.8 -> 106.5 mm
- net /SY3: track 118.3 -> 110.1 mm
- net /SY8: track 43.1 -> 38.0 mm
- net /~RY5: track 70.5 -> 75.0 mm
- net /~RY19: track 35.3 -> 37.6 mm
- net /~RY16: track 29.5 -> 31.3 mm
- net /~RY7: track 76.0 -> 77.7 mm
- net /~RY3: track 61.7 -> 60.3 mm
- net /SY18: track 55.4 -> 56.8 mm
- net /~RY20: track 25.5 -> 26.8 mm
- net /~RY15: track 28.5 -> 29.7 mm
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
Commit message: adding logo
Parts:
- added REF**: FlipsLogo-Mittel, Own:FlipsLogo-Mittel, F.Cu at (59.7, 78.7)
Changed lines of the file:
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@@
     (tracks 1038)
     (zones 0)
-    (modules 22)
+    (modules 23)
     (nets 158)
   )
@@
   )
   (layers
-    (0 F.Cu signal hide)
+    (0 F.Cu signal)
     (31 B.Cu signal)
     (32 B.Adhes user)
@@
     )
   )
+  (module Own:FlipsLogo-Mittel (layer F.Cu)
+    (at 59.69 78.74)
+    (fp_text reference REF** (at 0 3.81) (layer F.Fab) hide
+      (effects (font (size 1 1) (thickness 0.15)))
+    )
+    (fp_text value FlipsLogo-Mittel (at 0 2.54) (layer F.Fab)
+      (effects (font (size 1 1) (thickness 0.15)))
+    )
+    (fp_line (start -0.381 0) (end -0.6985 -0.3175) (layer F.SilkS) (width 0.2))
+    (fp_line (start -3.048 -2.667) (end -2.7178 -2.3368) (layer F.SilkS) (width 0.2))
+    (fp_line (start -3.048 1.778) (end -3.048 -2.667) (layer F.CrtYd) (width 0.1))
+    (fp_line (start 3.048 1.778) (end -3.048 1.778) (layer F.CrtYd) (width 0.1))
+    (fp_line (start 3.048 -2.667) (end 3.048 1.778) (layer F.CrtYd) (width 0.1))
+    (fp_line (start -3.048 -2.667) (end 3.048 -2.667) (layer F.CrtYd) (width 0.1))
+    (fp_poly (pts (xy -0.381 -1.905) (xy -0.381 -0.762) (xy -1.143 0) (xy -2.286 0)
+      (xy -3.048 -0.762) (xy -3.048 -1.905) (xy -2.286 -2.667) (xy -1.143 -2.667)) (layer F.SilkS) (width 0.15))
+    (fp_line (start 0.381 -2.667) (end 0.7112 -2.3368) (layer F.SilkS) (width 0.2))
+    (fp_line (start 1.143 0) (end 2.286 0) (layer F.SilkS) (width 0.1))
+    (fp_line (start 0.381 -0.762) (end 1.143 0) (layer F.SilkS) (width 0.1))
+    (fp_line (start 0.381 -1.905) (end 0.381 -0.762) (layer F.SilkS) (width 0.1))
+    (fp_line (start 1.143 -2.667) (end 0.381 -1.905) (layer F.SilkS) (width 0.1))
+    (fp_line (start 2.159 -2.667) (end 1.143 -2.667) (layer F.SilkS) (width 0.1))
+    (fp_line (start 3.048 -1.905) (end 2.286 -2.667) (layer F.SilkS) (width 0.1))
+    (fp_line (start 3.048 -0.762) (end 3.048 -1.905) (layer F.SilkS) (width 0.1))
+    (fp_line (start 2.286 0) (end 3.048 -0.762) (layer F.SilkS) (width 0.1))
+    (fp_line (start 3.048 0) (end 2.7305 -0.3175) (layer F.SilkS) (width 0.2))
+    (fp_text user FLIPS (at 0 1.016) (layer F.SilkS)
+      (effects (font (size 1 1) (thickness 0.2) italic))
+    )
+  )

Commit message: fixing missing VCC connection
Routing:
- net /VCC: track 58.6 -> 129.8 mm
- removed copper zone on F.Cu, net (none)
Changed lines of the file:
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@@
     (thickness 1.6)
     (drawings 110)
-    (tracks 1038)
+    (tracks 1050)
     (zones 0)
     (modules 23)
@@
     (uvia_dia 0.3)
     (uvia_drill 0.1)
+    (add_net /VCC)
     (add_net /X.A0)
     (add_net /X.A1)
@@
     (add_net /SY8)
     (add_net /SY9)
-    (add_net /VCC)
     (add_net /X1)
     (add_net /X10)
@@
   (segment (start 93.98 127) (end 96.54 127) (width 0.5) (layer F.Cu) (net 155) (status 30))
   (segment (start 99.06 142.24) (end 96.450006 139.630006) (width 0.2) (layer F.Cu) (net 155) (status 400010))
-  (segment (start 96.450006 127.089994) (end 96.54 127) (width 0.2) (layer F.Cu) (net 155) (status C00030))
   (segment (start 96.450006 139.630006) (end 96.450006 127.089994) (width 0.2) (layer F.Cu) (net 155) (status 800020))
+  (segment (start 96.450006 127.089994) (end 96.54 127) (width 0.2) (layer F.Cu) (net 155) (status C00030))
+  (segment (start 71.12 142.24) (end 69.85 143.51) (width 0.2) (layer B.Cu) (net 155) (status 400000))
+  (segment (start 97.79 143.51) (end 99.06 142.24) (width 0.2) (layer B.Cu) (net 155) (status 800000))
+  (segment (start 97.79 145.415) (end 97.79 143.51) (width 0.2) (layer B.Cu) (net 155))
+  (segment (start 95.25 147.955) (end 97.79 145.415) (width 0.2) (layer B.Cu) (net 155))
+  (segment (start 72.39 147.955) (end 95.25 147.955) (width 0.2) (layer B.Cu) (net 155))
+  (segment (start 69.85 145.415) (end 72.39 147.955) (width 0.2) (layer B.Cu) (net 155))
+  (segment (start 69.85 143.51) (end 69.85 145.415) (width 0.2) (layer B.Cu) (net 155))
+  (segment (start 97.79 145.415) (end 100.33 147.955) (width 0.2) (layer B.Cu) (net 155))
+  (segment (start 125.73 143.51) (end 127 142.24) (width 0.2) (layer B.Cu) (net 155) (status 800000))
+  (segment (start 125.73 145.415) (end 125.73 143.51) (width 0.2) (layer B.Cu) (net 155))
+  (segment (start 123.19 147.955) (end 125.73 145.415) (width 0.2) (layer B.Cu) (net 155))
+  (segment (start 100.33 147.955) (end 123.19 147.955) (width 0.2) (layer B.Cu) (net 155))
   (segment (start 127 126.98) (end 126.98 127) (width 0.5) (layer F.Cu) (net 156) (status 30))
   (via (at 127 128.905) (size 0.8) (drill 0.4) (layers F.Cu B.Cu) (net 156))
@@
   (segment (start 92.009998 95.59505) (end 92.009998 97.145098) (width 0.5) (layer F.Cu) (net 157))
   (segment (start 92.71 94.895048) (end 92.009998 95.59505) (width 0.5) (layer F.Cu) (net 157))
-  (zone (net 0) (net_name "") (layer F.Cu) (hatch edge 0.508)
+  (zone (net 156) (net_name /GND) (layer F.Cu) (hatch edge 0.508)
     (connect_pads (clearance 0.23))
     (min_thickness 0.254)
@@
     (polygon
       (pts
-        (xy 131.876 77.1585) (xy 131.826 77.5085) (xy 131.826 80.7085) (xy 128.826 80.7085) (xy 128.826 77.1585)
+        (xy 50.8 150.8) (xy 150.8 150.8) (xy 150.8 50.8) (xy 50.8 50.8)
       )
     )
   )
-  (zone (net 156) (net_name /GND) (layer F.Cu) (hatch edge 0.508)
+  (zone (net 156) (net_name /GND) (layer B.Cu) (hatch edge 0.508)
     (connect_pads (clearance 0.23))
     (min_thickness 0.254)
@@
     )
   )
-  (zone (net 156) (net_name /GND) (layer B.Cu) (hatch edge 0.508)
+  (zone (net 0) (net_name "") (layer F.Cu) (hatch edge 0.508)
     (connect_pads (clearance 0.23))
-    (min_thickness 0.254)
-    (fill yes (arc_segments 16) (thermal_gap 0.508) (thermal_bridge_width 0.508))
+    (min_thickness 0.2)
+    (keepout (tracks not_allowed) (vias not_allowed) (copperpour not_allowed))
+    (fill (arc_segments 16) (thermal_gap 0.23) (thermal_bridge_width 0.508))
     (polygon
       (pts
-        (xy 50.8 150.8) (xy 150.8 150.8) (xy 150.8 50.8) (xy 50.8 50.8)
+        (xy 128.9304 77.1906) (xy 131.9276 77.1398) (xy 131.8006 78.0796) (xy 131.8006 80.1116) (xy 131.8768 80.6704)
+        (xy 128.8542 80.7466) (xy 128.9304 79.502) (xy 128.8796 77.2922)
       )
     )

Commit message: Rename Flips6c description
Other:
- board text added: "Brose 60 and 34 Pin FlipDot Matrix Interface Adaptor"
- board text removed: "Brose 60 Pin FlipDot Matrix Interface Row Driver with Column Driver Port"
Changed lines of the file:
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@@
     (effects (font (size 1.5 1.5) (thickness 0.3)) (justify left))
   )
-  (gr_text "Brose 60 Pin FlipDot Matrix Interface Row Driver\nwith Column Driver Port" (at 55.88 135.255 90) (layer F.SilkS)
+  (gr_text "Brose 60 and 34 Pin FlipDot Matrix Interface Adaptor" (at 53.34 135.255 90) (layer F.SilkS)
     (effects (font (size 1.5 1.5) (thickness 0.3)) (justify left))
   )

Commit message: Rename U1/2/3 to IC1/2/3
Parts:
- renumbered U1 to IC1, U2 to IC2, U3 to IC3
Changed lines of the file:
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@@
   )
   (net 0 "")
-  (net 1 "Net-(U1-Pad1)")
-  (net 2 "Net-(U2-Pad1)")
-  (net 3 "Net-(U2-Pad2)")
-  (net 4 "Net-(U2-Pad3)")
-  (net 5 "Net-(U2-Pad4)")
-  (net 6 "Net-(U2-Pad5)")
-  (net 7 "Net-(U2-Pad6)")
-  (net 8 "Net-(U2-Pad26)")
-  (net 9 "Net-(U2-Pad27)")
-  (net 10 "Net-(U2-Pad8)")
-  (net 11 "Net-(U2-Pad28)")
-  (net 12 "Net-(U2-Pad9)")
-  (net 13 "Net-(U2-Pad29)")
-  (net 14 "Net-(U2-Pad10)")
-  (net 15 "Net-(U2-Pad30)")
-  (net 16 "Net-(U2-Pad31)")
-  (net 17 "Net-(U2-Pad32)")
-  (net 18 "Net-(U2-Pad33)")
+  (net 1 "Net-(IC1-Pad1)")
+  (net 2 "Net-(IC2-Pad1)")
+  (net 3 "Net-(IC2-Pad2)")
+  (net 4 "Net-(IC2-Pad3)")
+  (net 5 "Net-(IC2-Pad4)")
+  (net 6 "Net-(IC2-Pad5)")
+  (net 7 "Net-(IC2-Pad6)")
+  (net 8 "Net-(IC2-Pad26)")
+  (net 9 "Net-(IC2-Pad27)")
+  (net 10 "Net-(IC2-Pad8)")
+  (net 11 "Net-(IC2-Pad28)")
+  (net 12 "Net-(IC2-Pad9)")
+  (net 13 "Net-(IC2-Pad29)")
+  (net 14 "Net-(IC2-Pad10)")
+  (net 15 "Net-(IC2-Pad30)")
+  (net 16 "Net-(IC2-Pad31)")
+  (net 17 "Net-(IC2-Pad32)")
+  (net 18 "Net-(IC2-Pad33)")
   (net 19 /SY1)
   (net 20 /SY2)
@@
   (net 72 /X13)
   (net 73 /X11)
-  (net 74 "Net-(U3-Pad1)")
+  (net 74 "Net-(IC3-Pad1)")
   (net 75 /Y1.A2)
   (net 76 /Y1.A0)
@@
     (add_net "Net-(BRDB1-Pad33)")
     (add_net "Net-(BRDB1-Pad34)")
-    (add_net "Net-(U1-Pad1)")
-    (add_net "Net-(U2-Pad1)")
-    (add_net "Net-(U2-Pad10)")
-    (add_net "Net-(U2-Pad2)")
-    (add_net "Net-(U2-Pad26)")
-    (add_net "Net-(U2-Pad27)")
-    (add_net "Net-(U2-Pad28)")
-    (add_net "Net-(U2-Pad29)")
-    (add_net "Net-(U2-Pad3)")
-    (add_net "Net-(U2-Pad30)")
-    (add_net "Net-(U2-Pad31)")
-    (add_net "Net-(U2-Pad32)")
-    (add_net "Net-(U2-Pad33)")
-    (add_net "Net-(U2-Pad4)")
-    (add_net "Net-(U2-Pad5)")
-    (add_net "Net-(U2-Pad6)")
-    (add_net "Net-(U2-Pad8)")
-    (add_net "Net-(U2-Pad9)")
-    (add_net "Net-(U3-Pad1)")
+    (add_net "Net-(IC1-Pad1)")
+    (add_net "Net-(IC2-Pad1)")
+    (add_net "Net-(IC2-Pad10)")
+    (add_net "Net-(IC2-Pad2)")
+    (add_net "Net-(IC2-Pad26)")
+    (add_net "Net-(IC2-Pad27)")
+    (add_net "Net-(IC2-Pad28)")
+    (add_net "Net-(IC2-Pad29)")
+    (add_net "Net-(IC2-Pad3)")
+    (add_net "Net-(IC2-Pad30)")
+    (add_net "Net-(IC2-Pad31)")
+    (add_net "Net-(IC2-Pad32)")
+    (add_net "Net-(IC2-Pad33)")
+    (add_net "Net-(IC2-Pad4)")
+    (add_net "Net-(IC2-Pad5)")
+    (add_net "Net-(IC2-Pad6)")
+    (add_net "Net-(IC2-Pad8)")
+    (add_net "Net-(IC2-Pad9)")
+    (add_net "Net-(IC3-Pad1)")
   )
   (net_class POW ""
@@
     (descr "40-lead though-hole mounted DIP package, row spacing 15.24 mm (600 mils), Socket")
     (tags "THT DIP DIL PDIP 2.54mm 15.24mm 600mil Socket")
-    (fp_text reference U3 (at 7.62 -2.33) (layer F.SilkS)
+    (fp_text reference IC3 (at 7.62 -2.33) (layer F.SilkS)
       (effects (font (size 1 1) (thickness 0.15)))
     )
@@
       (net 40 /X.B0))
     (pad 1 thru_hole circle (at 0 0) (size 1.6 1.6) (drill 0.8) (layers *.Cu *.Mask)
-      (net 74 "Net-(U3-Pad1)"))
+      (net 74 "Net-(IC3-Pad1)"))
     (model ${KISYS3DMOD}/Housings_DIP.3dshapes/DIP-40_W15.24mm_Socket.wrl
       (at (xyz 0 0 0))
@@
     (descr "40-lead though-hole mounted DIP package, row spacing 15.24 mm (600 mils), Socket")
     (tags "THT DIP DIL PDIP 2.54mm 15.24mm 600mil Socket")
-    (fp_text reference U1 (at 7.62 -2.33) (layer F.SilkS)
+    (fp_text reference IC1 (at 7.62 -2.33) (layer F.SilkS)
       (effects (font (size 1 1) (thickness 0.15)))
     )
@@
       (net 80 /Y1.B0))
     (pad 1 thru_hole circle (at 0 0) (size 1.6 1.6) (drill 0.8) (layers *.Cu *.Mask)
-      (net 1 "Net-(U1-Pad1)"))
+      (net 1 "Net-(IC1-Pad1)"))
     (model ${KISYS3DMOD}/Socket_Strips.3dshapes/Socket_Strip_Straight_1x20_Pitch2.54mm.wrl
       (offset (xyz 0 -24.12999963760376 0))
@@
     (descr "40-lead though-hole mounted DIP package, row spacing 15.24 mm (600 mils), Socket")
     (tags "THT DIP DIL PDIP 2.54mm 15.24mm 600mil Socket")
-    (fp_text reference U2 (at 7.62 -2.33) (layer F.SilkS)
+    (fp_text reference IC2 (at 7.62 -2.33) (layer F.SilkS)
       (effects (font (size 1 1) (thickness 0.15)))
     )
@@
     )
     (pad 1 thru_hole circle (at 0 0) (size 1.6 1.6) (drill 0.8) (layers *.Cu *.Mask)
-      (net 2 "Net-(U2-Pad1)"))
+      (net 2 "Net-(IC2-Pad1)"))
     (pad 21 thru_hole oval (at 15.24 48.26) (size 1.6 1.6) (drill 0.8) (layers *.Cu *.Mask)
       (net 87 /Y2.B0))
     (pad 2 thru_hole oval (at 0 2.54) (size 1.6 1.6) (drill 0.8) (layers *.Cu *.Mask)
-      (net 3 "Net-(U2-Pad2)"))
+      (net 3 "Net-(IC2-Pad2)"))
     (pad 22 thru_hole oval (at 15.24 45.72) (size 1.6 1.6) (drill 0.8) (layers *.Cu *.Mask)
       (net 88 /Y2.B1))
     (pad 3 thru_hole oval (at 0 5.08) (size 1.6 1.6) (drill 0.8) (layers *.Cu *.Mask)
-      (net 4 "Net-(U2-Pad3)"))
+      (net 4 "Net-(IC2-Pad3)"))
     (pad 23 thru_hole oval (at 15.24 43.18) (size 1.6 1.6) (drill 0.8) (layers *.Cu *.Mask)
       (net 85 /Y2.POL))
     (pad 4 thru_hole oval (at 0 7.62) (size 1.6 1.6) (drill 0.8) (layers *.Cu *.Mask)
-      (net 5 "Net-(U2-Pad4)"))
+      (net 5 "Net-(IC2-Pad4)"))
     (pad 24 thru_hole oval (at 15.24 40.64) (size 1.6 1.6) (drill 0.8) (layers *.Cu *.Mask)
       (net 86 /Y2.EN))
     (pad 5 thru_hole oval (at 0 10.16) (size 1.6 1.6) (drill 0.8) (layers *.Cu *.Mask)
-      (net 6 "Net-(U2-Pad5)"))
+      (net 6 "Net-(IC2-Pad5)"))
     (pad 25 thru_hole oval (at 15.24 38.1) (size 1.6 1.6) (drill 0.8) (layers *.Cu *.Mask)
       (net 156 /GND))
     (pad 6 thru_hole oval (at 0 12.7) (size 1.6 1.6) (drill 0.8) (layers *.Cu *.Mask)
-      (net 7 "Net-(U2-Pad6)"))
+      (net 7 "Net-(IC2-Pad6)"))
     (pad 26 thru_hole oval (at 15.24 35.56) (size 1.6 1.6) (drill 0.8) (layers *.Cu *.Mask)
-      (net 8 "Net-(U2-Pad26)"))
+      (net 8 "Net-(IC2-Pad26)"))
     (pad 7 thru_hole oval (at 0 15.24) (size 1.6 1.6) (drill 0.8) (layers *.Cu *.Mask)
       (net 156 /GND))
     (pad 27 thru_hole oval (at 15.24 33.02) (size 1.6 1.6) (drill 0.8) (layers *.Cu *.Mask)
-      (net 9 "Net-(U2-Pad27)"))
+      (net 9 "Net-(IC2-Pad27)"))
     (pad 8 thru_hole oval (at 0 17.78) (size 1.6 1.6) (drill 0.8) (layers *.Cu *.Mask)
-      (net 10 "Net-(U2-Pad8)"))
+      (net 10 "Net-(IC2-Pad8)"))
     (pad 28 thru_hole oval (at 15.24 30.48) (size 1.6 1.6) (drill 0.8) (layers *.Cu *.Mask)
-      (net 11 "Net-(U2-Pad28)"))
+      (net 11 "Net-(IC2-Pad28)"))
     (pad 9 thru_hole oval (at 0 20.32) (size 1.6 1.6) (drill 0.8) (layers *.Cu *.Mask)
-      (net 12 "Net-(U2-Pad9)"))
+      (net 12 "Net-(IC2-Pad9)"))
     (pad 29 thru_hole oval (at 15.24 27.94) (size 1.6 1.6) (drill 0.8) (layers *.Cu *.Mask)
-      (net 13 "Net-(U2-Pad29)"))
+      (net 13 "Net-(IC2-Pad29)"))
     (pad 10 thru_hole oval (at 0 22.86) (size 1.6 1.6) (drill 0.8) (layers *.Cu *.Mask)
-      (net 14 "Net-(U2-Pad10)"))
+      (net 14 "Net-(IC2-Pad10)"))
     (pad 30 thru_hole oval (at 15.24 25.4) (size 1.6 1.6) (drill 0.8) (layers *.Cu *.Mask)
-      (net 15 "Net-(U2-Pad30)"))
+      (net 15 "Net-(IC2-Pad30)"))
     (pad 11 thru_hole oval (at 0 25.4) (size 1.6 1.6) (drill 0.8) (layers *.Cu *.Mask)
       (net 37 /SY19))
     (pad 31 thru_hole oval (at 15.24 22.86) (size 1.6 1.6) (drill 0.8) (layers *.Cu *.Mask)
-      (net 16 "Net-(U2-Pad31)"))
+      (net 16 "Net-(IC2-Pad31)"))
     (pad 12 thru_hole oval (at 0 27.94) (size 1.6 1.6) (drill 0.8) (layers *.Cu *.Mask)
       (net 38 /SY20))
     (pad 32 thru_hole oval (at 15.24 20.32) (size 1.6 1.6) (drill 0.8) (layers *.Cu *.Mask)
-      (net 17 "Net-(U2-Pad32)"))
+      (net 17 "Net-(IC2-Pad32)"))
     (pad 13 thru_hole oval (at 0 30.48) (size 1.6 1.6) (drill 0.8) (layers *.Cu *.Mask)
       (net 36 /SY18))
     (pad 33 thru_hole oval (at 15.24 17.78) (size 1.6 1.6) (drill 0.8) (layers *.Cu *.Mask)
-      (net 18 "Net-(U2-Pad33)"))
+      (net 18 "Net-(IC2-Pad33)"))
     (pad 14 thru_hole oval (at 0 33.02) (size 1.6 1.6) (drill 0.8) (layers *.Cu *.Mask)
       (net 35 /SY17))
