File: Flips5/Flips5.sch (KiCad schematic (older format))
At the start: 3 parts, among them CN1 Conn_02x30_Odd_Even, CN2 FP2800A, CN3 FP2800A

Commit message: moving abandoned project, renaming remaining
Parts:
- added BRDA2, BRDB1: Conn_02x17_Odd_Even, Own:Pin_Header_Angle_Shrouded_2x17_Pitch2.54mm_ConvNumbering, symbol Connector_Generic:Conn_02x17_Odd_Even
- added C1, C2, C3: 0μ1, Capacitors_SMD:C_0805_HandSoldering, symbol Device:C_Small
- added CNX1, CNY1, CNY2: UFP2810, Own:Pin_Header_Angle_Shrouded_2x05_Pitch2.54mm, symbol Eigene~Bauteile:UFP2810
- added IC3: FP2800A, Housings_DIP:DIP-40_W15.24mm_Socket, symbol Eigene~Bauteile:FP2800A
- added R1, R2, R3: 10k, Resistors_SMD:R_0805_HandSoldering, symbol Device:R_Small
- BRDA1: renamed from CN1; footprint Socket_Strips:Socket_Strip_Straight_2x30_Pitch2.54mm -> Own:Pin_Header_Straight_Shrouded_2x30_Pitch2.54mm_ConvNumbering
- IC1: renamed from CN2; footprint Own:DIP-32-from-40_W15.24mm -> Housings_DIP:DIP-40_W15.24mm_Socket
- IC2: renamed from CN3; footprint Own:DIP-32-from-40_W15.24mm -> Housings_DIP:DIP-40_W15.24mm_Socket
Connections:
- net labels added: GND, HV, SY1, SY10, SY11, SY12, SY13, SY14, SY15, SY16, SY17, SY18, SY19, SY2, SY20, SY3, SY4, SY5, SY6, SY7, SY8, SY9, VCC, X.A0, X.A1, X.A2, X.B0, X.B1, X.EN, X.POL, X1, X10, X11, X12, X13, X14, X15, X16, X17, X18, X19, X2, X20, X21, X22, X23, X24, X25, X26, X27, X28, X3, X4, X5, X6, X7, X8, X9, Y1.A0, Y1.A1, Y1.A2, Y1.B0, Y1.B1, Y1.EN, Y1.POL, Y2.A0, Y2.A1, Y2.A2, Y2.B0, Y2.B1, Y2.EN, Y2.POL, ~RY1, ~RY10, ~RY11, ~RY12, ~RY13, ~RY14, ~RY15, ~RY16, ~RY17, ~RY18, ~RY19, ~RY2, ~RY20, ~RY3, ~RY4, ~RY5, ~RY6, ~RY7, ~RY8, ~RY9
- wire segments 120 -> 6
- no-connect marks 60 -> 65
Other:
- moved on the sheet: BRDA1
