File: Flips5/Flips5.sch (KiCad schematic (older format))
At the start: 15 parts, among them IC1 FP2800A, IC2 FP2800A, IC3 FP2800A

Commit message: Adding Rows 21-28 (extra connector; preliminary pin assignment)
Parts:
- added BRDA3: Conn_02x10_Odd_Even, Own:Pin_Header_Straight_Shrouded_2x10_Pitch2.54mm_ConvNumbering, symbol Connector_Generic:Conn_02x10_Odd_Even
Connections:
- net labels added: SY21, SY22, SY23, SY24, SY25, SY26, SY27, SY28, ~RY21, ~RY22, ~RY23, ~RY24, ~RY25, ~RY26, ~RY27, ~RY28
- no-connect marks 65 -> 53
Changed lines of the file:
@@
 EESchema Schematic File Version 4
-LIBS:Flips5-cache
 EELAYER 26 0
 EELAYER END
@@
 NoConn ~ 5550 1500
 NoConn ~ 4250 3050
-NoConn ~ 7200 3150
-NoConn ~ 7300 3150
-NoConn ~ 7400 3150
-NoConn ~ 7500 3150
-NoConn ~ 7600 3150
-NoConn ~ 7700 3150
-NoConn ~ 7800 3150
-NoConn ~ 8000 3150
-NoConn ~ 8800 3150
-NoConn ~ 8900 3150
-NoConn ~ 9000 3150
-NoConn ~ 9100 3150
-NoConn ~ 9200 3150
-NoConn ~ 9300 3150
-NoConn ~ 9400 3150
-NoConn ~ 9600 3150
 NoConn ~ 10400 3150
 $Comp
@@
 Text Label 9850 900  0    50   ~ 0
 GND
+$Comp
+L Connector_Generic:Conn_02x10_Odd_Even BRDA3
+U 1 1 5BF467D4
+P 4750 4000
+F 0 "BRDA3" H 4800 3275 50  0000 C CNN
+F 1 "Conn_02x10_Odd_Even" H 4800 3366 50  0000 C CNN
+F 2 "Own:Pin_Header_Straight_Shrouded_2x10_Pitch2.54mm_ConvNumbering" H 4750 4000 50  0001 C CNN
+F 3 "~" H 4750 4000 50  0001 C CNN
+	1    4750 4000
+	-1   0    0    1
+$EndComp
+Text Label 4950 4400 0    50   ~ 0
+SY21
+Text Label 4450 4400 2    50   ~ 0
+SY22
+Text Label 4950 4300 0    50   ~ 0
+SY23
+Text Label 4950 4200 0    50   ~ 0
+SY25
+Text Label 4950 4100 0    50   ~ 0
+SY27
+Text Label 4450 4300 2    50   ~ 0
+SY24
+Text Label 4450 4200 2    50   ~ 0
+SY26
+Text Label 4450 4100 2    50   ~ 0
+SY28
+Text Label 4950 4000 0    50   ~ 0
+~RY21
+Text Label 4450 4000 2    50   ~ 0
+~RY22
+Text Label 4450 3900 2    50   ~ 0
+~RY24
+Text Label 4450 3800 2    50   ~ 0
+~RY26
+Text Label 4450 3700 2    50   ~ 0
+~RY28
+Text Label 4950 3900 0    50   ~ 0
+~RY23
+Text Label 4950 3800 0    50   ~ 0
+~RY25
+Text Label 4950 3700 0    50   ~ 0
+~RY27
+NoConn ~ 4950 3600
+NoConn ~ 4950 3500
+NoConn ~ 4450 3600
+NoConn ~ 4450 3500
+Text Label 9600 3150 3    50   ~ 0
+SY21
+Text Label 9400 3150 3    50   ~ 0
+SY22
+Text Label 9300 3150 3    50   ~ 0
+SY23
+Text Label 9200 3150 3    50   ~ 0
+SY24
+Text Label 9100 3150 3    50   ~ 0
+SY25
+Text Label 9000 3150 3    50   ~ 0
+SY26
+Text Label 8900 3150 3    50   ~ 0
+SY27
+Text Label 8800 3150 3    50   ~ 0
+SY28
+Text Label 8000 3150 3    50   ~ 0
+~RY21
+Text Label 7800 3150 3    50   ~ 0
+~RY22
+Text Label 7700 3150 3    50   ~ 0
+~RY23
+Text Label 7600 3150 3    50   ~ 0
+~RY24
+Text Label 7500 3150 3    50   ~ 0
+~RY25
+Text Label 7400 3150 3    50   ~ 0
+~RY26
+Text Label 7300 3150 3    50   ~ 0
+~RY27
+Text Label 7200 3150 3    50   ~ 0
+~RY28
 $EndSCHEMATC

Commit message: renaming connectors
Parts:
- renumbered BRDB1 to BRDIC1, BRDA3 to BROSE20, BRDA2 to BROSE34, BRDA1 to BROSE60
Changed lines of the file:
@@
 NoConn ~ 6100 5900
 $Comp
-L Connector_Generic:Conn_02x17_Odd_Even BRDB1
+L Connector_Generic:Conn_02x17_Odd_Even BRDIC1
 U 1 1 5BE36D58
 P 6900 5600
-F 0 "BRDB1" V 6996 6479 50  0000 L CNN
+F 0 "BRDIC1" V 6996 6479 50  0000 L CNN
 F 1 "Conn_02x17_Odd_Even" V 6905 6479 50  0000 L CNN
 F 2 "Own:Pin_Header_Angle_Shrouded_2x17_Pitch2.54mm_ConvNumbering" H 6900 5600 50  0001 C CNN
@@
 NoConn ~ 7700 5400
 $Comp
-L Connector_Generic:Conn_02x17_Odd_Even BRDA2
+L Connector_Generic:Conn_02x17_Odd_Even BROSE34
 U 1 1 5BE3715E
 P 7250 4450
-F 0 "BRDA2" V 7254 5329 50  0000 L CNN
+F 0 "BROSE34" V 7254 5329 50  0000 L CNN
 F 1 "Conn_02x17_Odd_Even" V 7345 5329 50  0000 L CNN
 F 2 "Own:Pin_Header_Angle_Shrouded_2x17_Pitch2.54mm_ConvNumbering" H 7250 4450 50  0001 C CNN
@@
 NoConn ~ 6550 4150
 $Comp
-L Connector_Generic:Conn_02x30_Odd_Even BRDA1
+L Connector_Generic:Conn_02x30_Odd_Even BROSE60
 U 1 1 5B82C747
 P 5850 2100
-F 0 "BRDA1" V 5500 1300 50  0000 C CNN
+F 0 "BROSE60" V 5500 1300 50  0000 C CNN
 F 1 "Conn_02x30_Odd_Even" V 6300 1050 50  0000 C CNN
 F 2 "Own:Pin_Header_Straight_Shrouded_2x30_Pitch2.54mm_ConvNumbering" H 5850 2100 50  0001 C CNN
@@
 GND
 $Comp
-L Connector_Generic:Conn_02x10_Odd_Even BRDA3
+L Connector_Generic:Conn_02x10_Odd_Even BROSE20
 U 1 1 5BF467D4
 P 4750 4000
-F 0 "BRDA3" H 4800 3275 50  0000 C CNN
+F 0 "BROSE20" H 4800 3275 50  0000 C CNN
 F 1 "Conn_02x10_Odd_Even" H 4800 3366 50  0000 C CNN
 F 2 "Own:Pin_Header_Straight_Shrouded_2x10_Pitch2.54mm_ConvNumbering" H 4750 4000 50  0001 C CNN
