File: Flips6/Flips6.sch (KiCad schematic (older format))
At the start: 17 parts, among them CN1 Conn_02x04_Odd_Even, IC1 74595, IC2 74595, IC3 74595

Commit message: fix footprint of 74595 to SOIC-16_3.9x9.9mm_Pitch1.27mm
Parts:
- IC1, IC2, IC3: footprint SMD_Packages:SO-16-N -> SOIC-16_3.9x9.9mm_Pitch1.27mm
Changed lines of the file:
@@
 EESchema Schematic File Version 4
-LIBS:Flips6-cache
 EELAYER 26 0
 EELAYER END
@@
 F 0 "IC1" H 1800 3500 50  0000 C CNN
 F 1 "74595" H 1950 3400 50  0000 C CNN
-F 2 "SMD_Packages:SO-16-N" H 1700 2800 50  0001 C CNN
+F 2 "SOIC-16_3.9x9.9mm_Pitch1.27mm" H 1700 2800 50  0001 C CNN
 F 3 "https://assets.nexperia.com/documents/data-sheet/74HC_HCT595.pdf" H 1700 2800 50  0001 C CNN
 	1    1700 2800
@@
 F 0 "IC2" H 3350 3500 50  0000 C CNN
 F 1 "74595" H 3500 3400 50  0000 C CNN
-F 2 "SMD_Packages:SO-16-N" H 3250 2800 50  0001 C CNN
+F 2 "SOIC-16_3.9x9.9mm_Pitch1.27mm" H 3250 2800 50  0001 C CNN
 F 3 "https://assets.nexperia.com/documents/data-sheet/74HC_HCT595.pdf" H 3250 2800 50  0001 C CNN
 	1    3250 2800
@@
 F 0 "IC3" H 4900 3500 50  0000 C CNN
 F 1 "74595" H 5050 3400 50  0000 C CNN
-F 2 "SMD_Packages:SO-16-N" H 4800 2800 50  0001 C CNN
+F 2 "SOIC-16_3.9x9.9mm_Pitch1.27mm" H 4800 2800 50  0001 C CNN
 F 3 "https://assets.nexperia.com/documents/data-sheet/74HC_HCT595.pdf" H 4800 2800 50  0001 C CNN
 	1    4800 2800

Commit message: adding pulldowns for enable pins
Parts:
- added R10, R3, R4, R5, R6, R7, R8, R9: 10k, Resistors_SMD:R_0805_HandSoldering, symbol Device:R_Small
Changed lines of the file:
@@
 EESchema Schematic File Version 4
+LIBS:Flips6-cache
 EELAYER 26 0
 EELAYER END
@@
 	1    0    0    1
 $EndComp
+Text Label 6450 850  2    50   ~ 0
+YEN1
+Text Label 6450 1100 2    50   ~ 0
+YEN2
+Text Label 6450 1350 2    50   ~ 0
+XEN1
+Text Label 6450 1600 2    50   ~ 0
+XEN2
+Text Label 6450 1850 2    50   ~ 0
+XEN3
+Text Label 6450 2100 2    50   ~ 0
+XEN4
+Text Label 6450 2350 2    50   ~ 0
+XEN5
+Text Label 6450 2600 2    50   ~ 0
+XEN6
+$Comp
+L Device:R_Small R3
+U 1 1 5BF7311F
+P 6550 850
+F 0 "R3" V 6450 900 50  0000 L CNN
+F 1 "10k" V 6450 700 50  0000 L CNN
+F 2 "Resistors_SMD:R_0805_HandSoldering" H 6550 850 50  0001 C CNN
+F 3 "~" H 6550 850 50  0001 C CNN
+	1    6550 850
+	0    1    1    0
+$EndComp
+$Comp
+L Device:R_Small R4
+U 1 1 5BF7321F
+P 6550 1100
+F 0 "R4" V 6450 1150 50  0000 L CNN
+F 1 "10k" V 6450 950 50  0000 L CNN
+F 2 "Resistors_SMD:R_0805_HandSoldering" H 6550 1100 50  0001 C CNN
+F 3 "~" H 6550 1100 50  0001 C CNN
+	1    6550 1100
+	0    1    1    0
+$EndComp
+$Comp
+L Device:R_Small R5
+U 1 1 5BF73255
+P 6550 1350
+F 0 "R5" V 6450 1400 50  0000 L CNN
+F 1 "10k" V 6450 1200 50  0000 L CNN
+F 2 "Resistors_SMD:R_0805_HandSoldering" H 6550 1350 50  0001 C CNN
+F 3 "~" H 6550 1350 50  0001 C CNN
+	1    6550 1350
+	0    1    1    0
+$EndComp
+$Comp
+L Device:R_Small R6
+U 1 1 5BF7328D
+P 6550 1600
+F 0 "R6" V 6450 1650 50  0000 L CNN
+F 1 "10k" V 6450 1450 50  0000 L CNN
+F 2 "Resistors_SMD:R_0805_HandSoldering" H 6550 1600 50  0001 C CNN
+F 3 "~" H 6550 1600 50  0001 C CNN
+	1    6550 1600
+	0    1    1    0
+$EndComp
+$Comp
+L Device:R_Small R7
+U 1 1 5BF732C7
+P 6550 1850
+F 0 "R7" V 6450 1900 50  0000 L CNN
+F 1 "10k" V 6450 1700 50  0000 L CNN
+F 2 "Resistors_SMD:R_0805_HandSoldering" H 6550 1850 50  0001 C CNN
+F 3 "~" H 6550 1850 50  0001 C CNN
+	1    6550 1850
+	0    1    1    0
+$EndComp
+$Comp
+L Device:R_Small R8
+U 1 1 5BF7332F
+P 6550 2100
+F 0 "R8" V 6450 2150 50  0000 L CNN
+F 1 "10k" V 6450 1950 50  0000 L CNN
+F 2 "Resistors_SMD:R_0805_HandSoldering" H 6550 2100 50  0001 C CNN
+F 3 "~" H 6550 2100 50  0001 C CNN
+	1    6550 2100
+	0    1    1    0
+$EndComp
+$Comp
+L Device:R_Small R9
+U 1 1 5BF7336D
+P 6550 2350
+F 0 "R9" V 6450 2400 50  0000 L CNN
+F 1 "10k" V 6450 2200 50  0000 L CNN
+F 2 "Resistors_SMD:R_0805_HandSoldering" H 6550 2350 50  0001 C CNN
+F 3 "~" H 6550 2350 50  0001 C CNN
+	1    6550 2350
+	0    1    1    0
+$EndComp
+$Comp
+L Device:R_Small R10
+U 1 1 5BF733AD
+P 6550 2600
+F 0 "R10" V 6450 2650 50  0000 L CNN
+F 1 "10k" V 6450 2450 50  0000 L CNN
+F 2 "Resistors_SMD:R_0805_HandSoldering" H 6550 2600 50  0001 C CNN
+F 3 "~" H 6550 2600 50  0001 C CNN
+	1    6550 2600
+	0    1    1    0
+$EndComp
+$Comp
+L power:GND #PWR07
+U 1 1 5BF73483
+P 6650 850
+F 0 "#PWR07" H 6650 600 50  0001 C CNN
+F 1 "GND" V 6655 722 50  0000 R CNN
+F 2 "" H 6650 850 50  0001 C CNN
+F 3 "" H 6650 850 50  0001 C CNN
+	1    6650 850
+	0    -1   -1   0
+$EndComp
+$Comp
+L power:GND #PWR018
+U 1 1 5BF73512
+P 6650 1100
+F 0 "#PWR018" H 6650 850 50  0001 C CNN
+F 1 "GND" V 6655 972 50  0000 R CNN
+F 2 "" H 6650 1100 50  0001 C CNN
+F 3 "" H 6650 1100 50  0001 C CNN
+	1    6650 1100
+	0    -1   -1   0
+$EndComp
+$Comp
+L power:GND #PWR019
+U 1 1 5BF7354F
+P 6650 1350
+F 0 "#PWR019" H 6650 1100 50  0001 C CNN
+F 1 "GND" V 6655 1222 50  0000 R CNN
+F 2 "" H 6650 1350 50  0001 C CNN
+F 3 "" H 6650 1350 50  0001 C CNN
+	1    6650 1350
+	0    -1   -1   0
+$EndComp
+$Comp
+L power:GND #PWR020
+U 1 1 5BF7358C
+P 6650 1600
+F 0 "#PWR020" H 6650 1350 50  0001 C CNN
+F 1 "GND" V 6655 1472 50  0000 R CNN
+F 2 "" H 6650 1600 50  0001 C CNN
+F 3 "" H 6650 1600 50  0001 C CNN
+	1    6650 1600
+	0    -1   -1   0
+$EndComp
+$Comp
+L power:GND #PWR021
+U 1 1 5BF735C9
+P 6650 1850
+F 0 "#PWR021" H 6650 1600 50  0001 C CNN
+F 1 "GND" V 6655 1722 50  0000 R CNN
+F 2 "" H 6650 1850 50  0001 C CNN
+F 3 "" H 6650 1850 50  0001 C CNN
+	1    6650 1850
+	0    -1   -1   0
+$EndComp
+$Comp
+L power:GND #PWR022
+U 1 1 5BF73606
+P 6650 2100
+F 0 "#PWR022" H 6650 1850 50  0001 C CNN
+F 1 "GND" V 6655 1972 50  0000 R CNN
+F 2 "" H 6650 2100 50  0001 C CNN
+F 3 "" H 6650 2100 50  0001 C CNN
+	1    6650 2100
+	0    -1   -1   0
+$EndComp
+$Comp
+L power:GND #PWR023
+U 1 1 5BF73643
+P 6650 2350
+F 0 "#PWR023" H 6650 2100 50  0001 C CNN
+F 1 "GND" V 6655 2222 50  0000 R CNN
+F 2 "" H 6650 2350 50  0001 C CNN
+F 3 "" H 6650 2350 50  0001 C CNN
+	1    6650 2350
+	0    -1   -1   0
+$EndComp
+$Comp
+L power:GND #PWR024
+U 1 1 5BF73680
+P 6650 2600
+F 0 "#PWR024" H 6650 2350 50  0001 C CNN
+F 1 "GND" V 6655 2472 50  0000 R CNN
+F 2 "" H 6650 2600 50  0001 C CNN
+F 3 "" H 6650 2600 50  0001 C CNN
+	1    6650 2600
+	0    -1   -1   0
+$EndComp
 $EndSCHEMATC
