File: Flips15/Group.sch (KiCad schematic (older format))
At the start: 6 parts, among them U301 74HC238, U302 ULN2803A, U303 74HC238, U304 TBD62783A

Commit message: rework Flips15 draft
Parts:
- U301, U303: footprint SMD_Packages:SO-16-N -> Housings_SOIC:SOIC-16_3.9x9.9mm_Pitch1.27mm
Connections:
- net ~GE is gone; now on net GND: U301.4 (~G2A), U303.4 (~G2A)
- net GND: now also U301.5 (~G2B)
- net VCC: no longer U301.6 (G1)
- net YH0: now reaches U303.15 (Y0), U304.1 (I1)
- net YH1: now reaches U303.14 (Y1), U304.2 (I2)
- net YH2: now reaches U303.13 (Y2), U304.3 (I3)
- net YH3: now reaches U303.12 (Y3), U304.4 (I4)
- net YH4: now reaches U303.11 (Y4), U304.5 (I5)
- net YH5: now reaches U303.10 (Y5), U304.6 (I6)
- net YH6: now reaches U303.9 (Y6), U304.7 (I7)
- net YH7: now reaches U303.7 (Y7), U304.8 (I8)
- net YL5: now reaches U301.10 (Y5), U302.6 (I6)
- net YL4: now reaches U301.11 (Y4), U302.5 (I5)
- net YL3: now reaches U301.12 (Y3), U302.4 (I4)
- net YL2: now reaches U301.13 (Y2), U302.3 (I3)
- net YL1: now reaches U301.14 (Y1), U302.2 (I2)
- net YL0: now reaches U301.15 (Y0), U302.1 (I1)
- net YL7: now reaches U301.7 (Y7), U302.8 (I8)
- net YL6: now reaches U301.9 (Y6), U302.7 (I7)
- net DATA renamed ENH
- net ENH: no longer U301.5 (~G2B)
- new net ENL: U301.6 (G1)

Commit message: Flips15 to only use 1 unit
Changed lines of the file:
@@
 $Descr A4 11693 8268
 encoding utf-8
-Sheet 8 11
+Sheet 8 6
 Title ""
 Date ""
@@
 AR Path="/5C4DA960/5C4DAAA8/5C4CE34D" Ref="U1004"  Part="1"
 AR Path="/5C4DA960/5C4DAABF/5C4CE34D" Ref="U1104"  Part="1"
-F 0 "U804" H 5900 4978 50  0000 C CNN
+F 0 "U1104" H 5900 4978 50  0000 C CNN
 F 1 "TBD62783A" H 5900 4887 50  0000 C CNN
 F 2 "Housings_DIP:DIP-18_W7.62mm_Socket" H 5900 3750 50  0001 C CNN
@@
 AR Path="/5C4DA960/5C4DAAA8/5C4CE354" Ref="U1001"  Part="1"
 AR Path="/5C4DA960/5C4DAABF/5C4CE354" Ref="U1101"  Part="1"
-F 0 "U801" H 4550 2116 50  0000 C CNN
+F 0 "U1101" H 4550 2116 50  0000 C CNN
 F 1 "74HC238" H 4550 2025 50  0000 C CNN
 F 2 "Housings_SOIC:SOIC-16_3.9x9.9mm_Pitch1.27mm" H 4550 1600 50  0001 C CNN
@@
 AR Path="/5C4DA960/5C4DAAA8/5C4CE35B" Ref="U1003"  Part="1"
 AR Path="/5C4DA960/5C4DAABF/5C4CE35B" Ref="U1103"  Part="1"
-F 0 "U803" H 4550 4716 50  0000 C CNN
+F 0 "U1103" H 4550 4716 50  0000 C CNN
 F 1 "74HC238" H 4550 4625 50  0000 C CNN
 F 2 "Housings_SOIC:SOIC-16_3.9x9.9mm_Pitch1.27mm" H 4550 4200 50  0001 C CNN
@@
 AR Path="/5C4DA960/5C4DAAA8/5C4D1DBE" Ref="#PWR01006"  Part="1"
 AR Path="/5C4DA960/5C4DAABF/5C4D1DBE" Ref="#PWR01106"  Part="1"
-F 0 "#PWR0806" H 5900 2350 50  0001 C CNN
+F 0 "#PWR01106" H 5900 2350 50  0001 C CNN
 F 1 "GND" H 5905 2427 50  0000 C CNN
 F 2 "" H 5900 2600 50  0001 C CNN
@@
 AR Path="/5C4DA960/5C4DAAA8/5C4D1DFA" Ref="#PWR01012"  Part="1"
 AR Path="/5C4DA960/5C4DAABF/5C4D1DFA" Ref="#PWR01112"  Part="1"
-F 0 "#PWR0812" H 5900 5050 50  0001 C CNN
+F 0 "#PWR01112" H 5900 5050 50  0001 C CNN
 F 1 "GND" H 5905 5127 50  0000 C CNN
 F 2 "" H 5900 5300 50  0001 C CNN
@@
 AR Path="/5C4DA960/5C4DAAA8/5C4D1E20" Ref="#PWR01011"  Part="1"
 AR Path="/5C4DA960/5C4DAABF/5C4D1E20" Ref="#PWR01111"  Part="1"
-F 0 "#PWR0811" H 4550 5050 50  0001 C CNN
+F 0 "#PWR01111" H 4550 5050 50  0001 C CNN
 F 1 "GND" H 4555 5127 50  0000 C CNN
 F 2 "" H 4550 5300 50  0001 C CNN
@@
 AR Path="/5C4DA960/5C4DAAA8/5C4D1E50" Ref="#PWR01005"  Part="1"
 AR Path="/5C4DA960/5C4DAABF/5C4D1E50" Ref="#PWR01105"  Part="1"
-F 0 "#PWR0805" H 4550 2350 50  0001 C CNN
+F 0 "#PWR01105" H 4550 2350 50  0001 C CNN
 F 1 "GND" H 4555 2427 50  0000 C CNN
 F 2 "" H 4550 2600 50  0001 C CNN
@@
 AR Path="/5C4DA960/5C4DAAA8/5C4D1F03" Ref="#PWR01002"  Part="1"
 AR Path="/5C4DA960/5C4DAABF/5C4D1F03" Ref="#PWR01102"  Part="1"
-F 0 "#PWR0802" H 6400 600 50  0001 C CNN
+F 0 "#PWR01102" H 6400 600 50  0001 C CNN
 F 1 "+24V" H 6415 923 50  0000 C CNN
 F 2 "" H 6400 750 50  0001 C CNN
@@
 AR Path="/5C4DA960/5C4DAAA8/5C4D1F1D" Ref="#PWR01008"  Part="1"
 AR Path="/5C4DA960/5C4DAABF/5C4D1F1D" Ref="#PWR01108"  Part="1"
-F 0 "#PWR0808" H 5900 3250 50  0001 C CNN
+F 0 "#PWR01108" H 5900 3250 50  0001 C CNN
 F 1 "+24V" H 5915 3573 50  0000 C CNN
 F 2 "" H 5900 3400 50  0001 C CNN
@@
 AR Path="/5C4DA960/5C4DAAA8/5C4D1FAA" Ref="#PWR01001"  Part="1"
 AR Path="/5C4DA960/5C4DAABF/5C4D1FAA" Ref="#PWR01101"  Part="1"
-F 0 "#PWR0801" H 4550 600 50  0001 C CNN
+F 0 "#PWR01101" H 4550 600 50  0001 C CNN
 F 1 "VCC" H 4567 923 50  0000 C CNN
 F 2 "" H 4550 750 50  0001 C CNN
@@
 AR Path="/5C4DA960/5C4DAAA8/5C4D1FD4" Ref="#PWR01007"  Part="1"
 AR Path="/5C4DA960/5C4DAABF/5C4D1FD4" Ref="#PWR01107"  Part="1"
-F 0 "#PWR0807" H 4550 3250 50  0001 C CNN
+F 0 "#PWR01107" H 4550 3250 50  0001 C CNN
 F 1 "VCC" H 4567 3573 50  0000 C CNN
 F 2 "" H 4550 3400 50  0001 C CNN
@@
 AR Path="/5C4DA960/5C4DAAA8/5C4DA0A7" Ref="#PWR01010"  Part="1"
 AR Path="/5C4DA960/5C4DAABF/5C4DA0A7" Ref="#PWR01110"  Part="1"
-F 0 "#PWR0810" H 3900 3900 50  0001 C CNN
+F 0 "#PWR01110" H 3900 3900 50  0001 C CNN
 F 1 "GND" V 3905 4022 50  0000 R CNN
 F 2 "" H 3900 4150 50  0001 C CNN
@@
 AR Path="/5C4DA960/5C4DAAA8/5C4E1AEA" Ref="U1002"  Part="1"
 AR Path="/5C4DA960/5C4DAABF/5C4E1AEA" Ref="U1102"  Part="1"
-F 0 "U802" H 5900 2167 50  0000 C CNN
+F 0 "U1102" H 5900 2167 50  0000 C CNN
 F 1 "ULN2803A" H 5900 2076 50  0000 C CNN
 F 2 "Housings_DIP:DIP-18_W7.62mm_Socket" H 5950 950 50  0001 L CNN
@@
 AR Path="/5C4DA960/5C4DAAA8/5C4F67EE" Ref="C1002"  Part="1"
 AR Path="/5C4DA960/5C4DAABF/5C4F67EE" Ref="C1102"  Part="1"
-F 0 "C802" V 4021 3500 50  0000 C CNN
+F 0 "C1102" V 4021 3500 50  0000 C CNN
 F 1 "0μ1" V 4112 3500 50  0000 C CNN
 F 2 "Capacitors_SMD:C_0805_HandSoldering" H 4250 3500 50  0001 C CNN
@@
 AR Path="/5C4DA960/5C4DAAA8/5C4F6885" Ref="C1001"  Part="1"
 AR Path="/5C4DA960/5C4DAABF/5C4F6885" Ref="C1101"  Part="1"
-F 0 "C801" V 4021 850 50  0000 C CNN
+F 0 "C1101" V 4021 850 50  0000 C CNN
 F 1 "0μ1" V 4112 850 50  0000 C CNN
 F 2 "Capacitors_SMD:C_0805_HandSoldering" H 4250 850 50  0001 C CNN
@@
 AR Path="/5C4DA960/5C4DAAA8/5C4F6943" Ref="#PWR01003"  Part="1"
 AR Path="/5C4DA960/5C4DAABF/5C4F6943" Ref="#PWR01103"  Part="1"
-F 0 "#PWR0803" H 3900 600 50  0001 C CNN
+F 0 "#PWR01103" H 3900 600 50  0001 C CNN
 F 1 "GND" V 3905 722 50  0000 R CNN
 F 2 "" H 3900 850 50  0001 C CNN
@@
 AR Path="/5C4DA960/5C4DAAA8/5C4F6978" Ref="#PWR01009"  Part="1"
 AR Path="/5C4DA960/5C4DAABF/5C4F6978" Ref="#PWR01109"  Part="1"
-F 0 "#PWR0809" H 3900 3250 50  0001 C CNN
+F 0 "#PWR01109" H 3900 3250 50  0001 C CNN
 F 1 "GND" V 3905 3372 50  0000 R CNN
 F 2 "" H 3900 3500 50  0001 C CNN
@@
 AR Path="/5C4DA960/5C4DAAA8/5C4EB0F4" Ref="#PWR0130"  Part="1"
 AR Path="/5C4DA960/5C4DAABF/5C4EB0F4" Ref="#PWR0133"  Part="1"
-F 0 "#PWR0124" H 3900 3750 50  0001 C CNN
+F 0 "#PWR0133" H 3900 3750 50  0001 C CNN
 F 1 "GND" V 3905 3872 50  0000 R CNN
 F 2 "" H 3900 4000 50  0001 C CNN
@@
 AR Path="/5C4DA960/5C4DAAA8/5C4EC62E" Ref="#PWR0131"  Part="1"
 AR Path="/5C4DA960/5C4DAABF/5C4EC62E" Ref="#PWR0134"  Part="1"
-F 0 "#PWR0125" H 3900 1150 50  0001 C CNN
+F 0 "#PWR0134" H 3900 1150 50  0001 C CNN
 F 1 "GND" V 3905 1272 50  0000 R CNN
 F 2 "" H 3900 1400 50  0001 C CNN
@@
 AR Path="/5C4DA960/5C4DAAA8/5C4EC645" Ref="#PWR0132"  Part="1"
 AR Path="/5C4DA960/5C4DAABF/5C4EC645" Ref="#PWR0135"  Part="1"
-F 0 "#PWR0126" H 3900 1300 50  0001 C CNN
+F 0 "#PWR0135" H 3900 1300 50  0001 C CNN
 F 1 "GND" V 3905 1422 50  0000 R CNN
 F 2 "" H 3900 1550 50  0001 C CNN

Commit message: Adding control wires - removing control for channel 0 - placing capacitor
Connections:
- net GND: now also U302.1 (I1), U304.1 (I1)
- net YH0: no longer names the net of U303.15 (Y0)
- net YH0: no longer U304.1 (I1)
- net YL0: no longer names the net of U301.15 (Y0)
- net YL0: no longer U302.1 (I1)
- no-connect marks 0 -> 2
Changed lines of the file:
@@
 $Descr A4 11693 8268
 encoding utf-8
-Sheet 8 6
+Sheet 3 6
 Title ""
 Date ""
@@
 AR Path="/5C4DA960/5C4DAAA8/5C4CE34D" Ref="U1004"  Part="1"
 AR Path="/5C4DA960/5C4DAABF/5C4CE34D" Ref="U1104"  Part="1"
-F 0 "U1104" H 5900 4978 50  0000 C CNN
+F 0 "U804" H 5900 4978 50  0000 C CNN
 F 1 "TBD62783A" H 5900 4887 50  0000 C CNN
 F 2 "Housings_DIP:DIP-18_W7.62mm_Socket" H 5900 3750 50  0001 C CNN
@@
 AR Path="/5C4DA960/5C4DAAA8/5C4CE354" Ref="U1001"  Part="1"
 AR Path="/5C4DA960/5C4DAABF/5C4CE354" Ref="U1101"  Part="1"
-F 0 "U1101" H 4550 2116 50  0000 C CNN
+F 0 "U801" H 4550 2116 50  0000 C CNN
 F 1 "74HC238" H 4550 2025 50  0000 C CNN
 F 2 "Housings_SOIC:SOIC-16_3.9x9.9mm_Pitch1.27mm" H 4550 1600 50  0001 C CNN
@@
 AR Path="/5C4DA960/5C4DAAA8/5C4CE35B" Ref="U1003"  Part="1"
 AR Path="/5C4DA960/5C4DAABF/5C4CE35B" Ref="U1103"  Part="1"
-F 0 "U1103" H 4550 4716 50  0000 C CNN
+F 0 "U803" H 4550 4716 50  0000 C CNN
 F 1 "74HC238" H 4550 4625 50  0000 C CNN
 F 2 "Housings_SOIC:SOIC-16_3.9x9.9mm_Pitch1.27mm" H 4550 4200 50  0001 C CNN
@@
 AR Path="/5C4DA960/5C4DAAA8/5C4D1DBE" Ref="#PWR01006"  Part="1"
 AR Path="/5C4DA960/5C4DAABF/5C4D1DBE" Ref="#PWR01106"  Part="1"
-F 0 "#PWR01106" H 5900 2350 50  0001 C CNN
+F 0 "#PWR0806" H 5900 2350 50  0001 C CNN
 F 1 "GND" H 5905 2427 50  0000 C CNN
 F 2 "" H 5900 2600 50  0001 C CNN
@@
 AR Path="/5C4DA960/5C4DAAA8/5C4D1DFA" Ref="#PWR01012"  Part="1"
 AR Path="/5C4DA960/5C4DAABF/5C4D1DFA" Ref="#PWR01112"  Part="1"
-F 0 "#PWR01112" H 5900 5050 50  0001 C CNN
+F 0 "#PWR0812" H 5900 5050 50  0001 C CNN
 F 1 "GND" H 5905 5127 50  0000 C CNN
 F 2 "" H 5900 5300 50  0001 C CNN
@@
 AR Path="/5C4DA960/5C4DAAA8/5C4D1E20" Ref="#PWR01011"  Part="1"
 AR Path="/5C4DA960/5C4DAABF/5C4D1E20" Ref="#PWR01111"  Part="1"
-F 0 "#PWR01111" H 4550 5050 50  0001 C CNN
+F 0 "#PWR0811" H 4550 5050 50  0001 C CNN
 F 1 "GND" H 4555 5127 50  0000 C CNN
 F 2 "" H 4550 5300 50  0001 C CNN
@@
 AR Path="/5C4DA960/5C4DAAA8/5C4D1E50" Ref="#PWR01005"  Part="1"
 AR Path="/5C4DA960/5C4DAABF/5C4D1E50" Ref="#PWR01105"  Part="1"
-F 0 "#PWR01105" H 4550 2350 50  0001 C CNN
+F 0 "#PWR0805" H 4550 2350 50  0001 C CNN
 F 1 "GND" H 4555 2427 50  0000 C CNN
 F 2 "" H 4550 2600 50  0001 C CNN
@@
 AR Path="/5C4DA960/5C4DAAA8/5C4D1F03" Ref="#PWR01002"  Part="1"
 AR Path="/5C4DA960/5C4DAABF/5C4D1F03" Ref="#PWR01102"  Part="1"
-F 0 "#PWR01102" H 6400 600 50  0001 C CNN
+F 0 "#PWR0802" H 6400 600 50  0001 C CNN
 F 1 "+24V" H 6415 923 50  0000 C CNN
 F 2 "" H 6400 750 50  0001 C CNN
@@
 AR Path="/5C4DA960/5C4DAAA8/5C4D1F1D" Ref="#PWR01008"  Part="1"
 AR Path="/5C4DA960/5C4DAABF/5C4D1F1D" Ref="#PWR01108"  Part="1"
-F 0 "#PWR01108" H 5900 3250 50  0001 C CNN
+F 0 "#PWR0808" H 5900 3250 50  0001 C CNN
 F 1 "+24V" H 5915 3573 50  0000 C CNN
 F 2 "" H 5900 3400 50  0001 C CNN
@@
 AR Path="/5C4DA960/5C4DAAA8/5C4D1FAA" Ref="#PWR01001"  Part="1"
 AR Path="/5C4DA960/5C4DAABF/5C4D1FAA" Ref="#PWR01101"  Part="1"
-F 0 "#PWR01101" H 4550 600 50  0001 C CNN
+F 0 "#PWR0801" H 4550 600 50  0001 C CNN
 F 1 "VCC" H 4567 923 50  0000 C CNN
 F 2 "" H 4550 750 50  0001 C CNN
@@
 AR Path="/5C4DA960/5C4DAAA8/5C4D1FD4" Ref="#PWR01007"  Part="1"
 AR Path="/5C4DA960/5C4DAABF/5C4D1FD4" Ref="#PWR01107"  Part="1"
-F 0 "#PWR01107" H 4550 3250 50  0001 C CNN
+F 0 "#PWR0807" H 4550 3250 50  0001 C CNN
 F 1 "VCC" H 4567 3573 50  0000 C CNN
 F 2 "" H 4550 3400 50  0001 C CNN
@@
 AR Path="/5C4DA960/5C4DAAA8/5C4DA0A7" Ref="#PWR01010"  Part="1"
 AR Path="/5C4DA960/5C4DAABF/5C4DA0A7" Ref="#PWR01110"  Part="1"
-F 0 "#PWR01110" H 3900 3900 50  0001 C CNN
+F 0 "#PWR0810" H 3900 3900 50  0001 C CNN
 F 1 "GND" V 3905 4022 50  0000 R CNN
 F 2 "" H 3900 4150 50  0001 C CNN
@@
 AR Path="/5C4DA960/5C4DAAA8/5C4E1AEA" Ref="U1002"  Part="1"
 AR Path="/5C4DA960/5C4DAABF/5C4E1AEA" Ref="U1102"  Part="1"
-F 0 "U1102" H 5900 2167 50  0000 C CNN
+F 0 "U802" H 5900 2167 50  0000 C CNN
 F 1 "ULN2803A" H 5900 2076 50  0000 C CNN
 F 2 "Housings_DIP:DIP-18_W7.62mm_Socket" H 5950 950 50  0001 L CNN
@@
 0L
 Wire Wire Line
-	5100 1400 5500 1400
-Wire Wire Line
 	6300 1400 7050 1400
 Wire Wire Line
@@
 Wire Wire Line
 	5900 3800 5900 3400
-Wire Wire Line
-	5100 4000 5500 4000
 Wire Wire Line
 	5900 4900 5900 5300
@@
 AR Path="/5C4DA960/5C4DAAA8/5C4F67EE" Ref="C1002"  Part="1"
 AR Path="/5C4DA960/5C4DAABF/5C4F67EE" Ref="C1102"  Part="1"
-F 0 "C1102" V 4021 3500 50  0000 C CNN
+F 0 "C802" V 4021 3500 50  0000 C CNN
 F 1 "0μ1" V 4112 3500 50  0000 C CNN
 F 2 "Capacitors_SMD:C_0805_HandSoldering" H 4250 3500 50  0001 C CNN
@@
 AR Path="/5C4DA960/5C4DAAA8/5C4F6885" Ref="C1001"  Part="1"
 AR Path="/5C4DA960/5C4DAABF/5C4F6885" Ref="C1101"  Part="1"
-F 0 "C1101" V 4021 850 50  0000 C CNN
+F 0 "C801" V 4021 850 50  0000 C CNN
 F 1 "0μ1" V 4112 850 50  0000 C CNN
 F 2 "Capacitors_SMD:C_0805_HandSoldering" H 4250 850 50  0001 C CNN
@@
 AR Path="/5C4DA960/5C4DAAA8/5C4F6943" Ref="#PWR01003"  Part="1"
 AR Path="/5C4DA960/5C4DAABF/5C4F6943" Ref="#PWR01103"  Part="1"
-F 0 "#PWR01103" H 3900 600 50  0001 C CNN
+F 0 "#PWR0803" H 3900 600 50  0001 C CNN
 F 1 "GND" V 3905 722 50  0000 R CNN
 F 2 "" H 3900 850 50  0001 C CNN
@@
 AR Path="/5C4DA960/5C4DAAA8/5C4F6978" Ref="#PWR01009"  Part="1"
 AR Path="/5C4DA960/5C4DAABF/5C4F6978" Ref="#PWR01109"  Part="1"
-F 0 "#PWR01109" H 3900 3250 50  0001 C CNN
+F 0 "#PWR0809" H 3900 3250 50  0001 C CNN
 F 1 "GND" V 3905 3372 50  0000 R CNN
 F 2 "" H 3900 3500 50  0001 C CNN
@@
 AR Path="/5C4DA960/5C4DAAA8/5C4EB0F4" Ref="#PWR0130"  Part="1"
 AR Path="/5C4DA960/5C4DAABF/5C4EB0F4" Ref="#PWR0133"  Part="1"
-F 0 "#PWR0133" H 3900 3750 50  0001 C CNN
+F 0 "#PWR0124" H 3900 3750 50  0001 C CNN
 F 1 "GND" V 3905 3872 50  0000 R CNN
 F 2 "" H 3900 4000 50  0001 C CNN
@@
 AR Path="/5C4DA960/5C4DAAA8/5C4EC62E" Ref="#PWR0131"  Part="1"
 AR Path="/5C4DA960/5C4DAABF/5C4EC62E" Ref="#PWR0134"  Part="1"
-F 0 "#PWR0134" H 3900 1150 50  0001 C CNN
+F 0 "#PWR0125" H 3900 1150 50  0001 C CNN
 F 1 "GND" V 3905 1272 50  0000 R CNN
 F 2 "" H 3900 1400 50  0001 C CNN
@@
 AR Path="/5C4DA960/5C4DAAA8/5C4EC645" Ref="#PWR0132"  Part="1"
 AR Path="/5C4DA960/5C4DAABF/5C4EC645" Ref="#PWR0135"  Part="1"
-F 0 "#PWR0135" H 3900 1300 50  0001 C CNN
+F 0 "#PWR0126" H 3900 1300 50  0001 C CNN
 F 1 "GND" V 3905 1422 50  0000 R CNN
 F 2 "" H 3900 1550 50  0001 C CNN
@@
 Wire Wire Line
 	3900 1400 4000 1400
-Text Label 5150 1400 0    50   ~ 0
-YL0
 Text Label 5150 1500 0    50   ~ 0
 YL1
@@
 Text Label 5150 2100 0    50   ~ 0
 YL7
-Text Label 5150 4000 0    50   ~ 0
-YH0
 Text Label 5150 4100 0    50   ~ 0
 YH1
@@
 Text Label 5150 4700 0    50   ~ 0
 YH7
+NoConn ~ 5100 1400
+NoConn ~ 5100 4000
+$Comp
+L power:GND #PWR?
+U 1 1 5C57C882
+P 5500 1400
+F 0 "#PWR?" H 5500 1150 50  0001 C CNN
+F 1 "GND" V 5505 1272 50  0000 R CNN
+F 2 "" H 5500 1400 50  0001 C CNN
+F 3 "" H 5500 1400 50  0001 C CNN
+	1    5500 1400
+	0    1    1    0
+$EndComp
+$Comp
+L power:GND #PWR?
+U 1 1 5C57C8A6
+P 5500 4000
+F 0 "#PWR?" H 5500 3750 50  0001 C CNN
+F 1 "GND" V 5505 3872 50  0000 R CNN
+F 2 "" H 5500 4000 50  0001 C CNN
+F 3 "" H 5500 4000 50  0001 C CNN
+	1    5500 4000
+	0    1    1    0
+$EndComp
 $EndSCHEMATC

Commit message: more silk screen (use more compact IC values)
Parts:
- U301, U303: value 74HC238 -> 74238
- U302: value ULN2803A -> ULN2803/2003
- U304: value TBD62783A -> TD62783
Changed lines of the file:
@@
 AR Path="/5C4DA960/5C4DAABF/5C4CE34D" Ref="U1104"  Part="1"
 F 0 "U804" H 5900 4978 50  0000 C CNN
-F 1 "TBD62783A" H 5900 4887 50  0000 C CNN
+F 1 "TD62783" H 5900 4887 50  0000 C CNN
 F 2 "Housings_DIP:DIP-18_W7.62mm_Socket" H 5900 3750 50  0001 C CNN
 F 3 "http://toshiba.semicon-storage.com/info/docget.jsp?did=30523&prodName=TBD62783APG" H 5600 4700 50  0001 C CNN
@@
 AR Path="/5C4DA960/5C4DAABF/5C4CE354" Ref="U1101"  Part="1"
 F 0 "U801" H 4550 2116 50  0000 C CNN
-F 1 "74HC238" H 4550 2025 50  0000 C CNN
+F 1 "74238" H 4550 2025 50  0000 C CNN
 F 2 "Housings_SOIC:SOIC-16_3.9x9.9mm_Pitch1.27mm" H 4550 1600 50  0001 C CNN
 F 3 "" H 4550 1600 50  0001 C CNN
@@
 AR Path="/5C4DA960/5C4DAABF/5C4CE35B" Ref="U1103"  Part="1"
 F 0 "U803" H 4550 4716 50  0000 C CNN
-F 1 "74HC238" H 4550 4625 50  0000 C CNN
+F 1 "74238" H 4550 4625 50  0000 C CNN
 F 2 "Housings_SOIC:SOIC-16_3.9x9.9mm_Pitch1.27mm" H 4550 4200 50  0001 C CNN
 F 3 "" H 4550 4200 50  0001 C CNN
@@
 AR Path="/5C4DA960/5C4DAABF/5C4E1AEA" Ref="U1102"  Part="1"
 F 0 "U802" H 5900 2167 50  0000 C CNN
-F 1 "ULN2803A" H 5900 2076 50  0000 C CNN
+F 1 "ULN2803/2003" H 5900 2076 50  0000 C CNN
 F 2 "Housings_DIP:DIP-18_W7.62mm_Socket" H 5950 950 50  0001 L CNN
 F 3 "http://www.ti.com/lit/ds/symlink/uln2803a.pdf" H 6000 1400 50  0001 C CNN
@@
 U 1 1 5C57C882
 P 5500 1400
+AR Path="/5C4DA960/5C4DAA7A/5C57C882" Ref="#PWR?"  Part="1"
+AR Path="/5C4DA960/5C4DAA91/5C57C882" Ref="#PWR?"  Part="1"
+AR Path="/5C4DA960/5C4DAAA8/5C57C882" Ref="#PWR?"  Part="1"
+AR Path="/5C4DA960/5C4DAABF/5C57C882" Ref="#PWR?"  Part="1"
 F 0 "#PWR?" H 5500 1150 50  0001 C CNN
 F 1 "GND" V 5505 1272 50  0000 R CNN
@@
 U 1 1 5C57C8A6
 P 5500 4000
+AR Path="/5C4DA960/5C4DAA7A/5C57C8A6" Ref="#PWR?"  Part="1"
+AR Path="/5C4DA960/5C4DAA91/5C57C8A6" Ref="#PWR?"  Part="1"
+AR Path="/5C4DA960/5C4DAAA8/5C57C8A6" Ref="#PWR?"  Part="1"
+AR Path="/5C4DA960/5C4DAABF/5C57C8A6" Ref="#PWR?"  Part="1"
 F 0 "#PWR?" H 5500 3750 50  0001 C CNN
 F 1 "GND" V 5505 3872 50  0000 R CNN
