File: Flips10/Flips10Base/Flips10Base.kicad_pcb (KiCad board)
At the start: 2 copper layers, 21.6 x 41.3 mm, 44 parts, among them U1 74138, U11 74238, U12 74238, U13 ULN2803/2003, U14 TD62783, U15 741G04, U21 74238, U22 74238, U23 ULN2803/2003, U24 TD62783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

Commit message: progress for flips10 base
Parts:
- removed C11, C12, C13, C21, C22, C23, C31, C32, C33, C41, C42, C43: 0μ1, Capacitors_SMD:C_0805_HandSoldering
- removed JP11, JP12, JP21, JP22, JP31, JP32, JP41, JP42: Jumper, Own:SolderJumper1.3mmChoice
- removed REF**: Pin_Header_Angled_2x08_Pitch2.54mm, Pin_Headers:Pin_Header_Angled_2x08_Pitch2.54mm
- removed U1: 74138, Housings_SOIC:SOIC-16_3.9x9.9mm_Pitch1.27mm
- removed U11, U12, U21, U22, U31, U32, U41, U42: 74238, Housings_SOIC:SOIC-16_3.9x9.9mm_Pitch1.27mm
- removed U13, U23, U33, U43: ULN2803/2003, Housings_SOIC:SOIC-18W_7.5x11.6mm_Pitch1.27mm
- removed U14, U24, U34, U44: TD62783, Own:SOP18
- removed U15, U25, U35, U45: 741G04, TO_SOT_Packages_SMD:SOT-23-5
- added CN0: SR28GR, Socket_Strips:Socket_Strip_Straight_2x08_Pitch2.54mm, F.Cu at (59.1, 73.7)
- added CN1: SR28GR, Socket_Strips:Socket_Strip_Straight_2x08_Pitch2.54mm, F.Cu at (59.1, 52.1)
- added CN2: SR28GR, Socket_Strips:Socket_Strip_Straight_2x08_Pitch2.54mm, F.Cu at (65.4, 53.0)
- added CN3: SR28GR, Socket_Strips:Socket_Strip_Straight_2x08_Pitch2.54mm, F.Cu at (65.4, 73.3)
- added IC1: 74138, Housings_SOIC:SOIC-16_3.9x9.9mm_Pitch1.27mm, F.Cu at (61.0, 96.5)
- C1: moved to B.Cu
- S1: value FP2800A -> FP2800A-Interface; footprint Housings_DIP:DIP-40_W15.24mm_Socket -> Housings_DIP:DIP-40_W15.24mm
- moved C1 167.9 mm to (56.5, 95.2), turned to 270 degrees
- moved S1 128.6 mm to (53.3, 51.7)
Routing:
- net /A2: track 10.5 -> 90.1 mm, vias 1 -> 4
- net GND: track 13.2 -> 84.3 mm, vias 0 -> 2
- net /DATA: track 6.53 -> 73.5 mm, vias 1 -> 0
- net VCC: track 2.24 -> 61.7 mm, vias 0 -> 1
- net /A1: track 11.4 -> 68.3 mm, vias 1 -> 3
- net /~ENGR1: track 0.00 -> 56.9 mm
- net +24V: track 0.00 -> 53.9 mm, vias 0 -> 2
- net /~ENGR2: track 0.00 -> 48.3 mm
- net /A0: track 14.3 -> 61.1 mm, vias 1 -> 3
- net /~ENGR3: track 0.00 -> 30.5 mm
- net /2G: track 0.00 -> 25.6 mm
- net /1G: track 0.00 -> 25.1 mm
- net /UnitY/Group0/YL7: track 23.7 -> 0.00 mm
- net /~ENGR0: track 0.00 -> 22.2 mm
- net /1E: track 0.00 -> 19.2 mm
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Other:
- board size 21.6 x 41.3 mm -> 20 x 50 mm
